File: hw/sch_pcb/USTSIPM01A.kicad_pcb (KiCad board)
At the start: 2 copper layers, 30 x 40.1 mm, 39 parts, among them J1 HEADER_2x01_PARALLEL, J10 HEADER_2x01_PARALLEL, J2 HEADER_2x01_PARALLEL, J3 HEADER_2x01_PARALLEL, J4 HEADER_2x01_PARALLEL, J5 HEADER_2x01_PARALLEL, J6 HEADER_2x01_PARALLEL, J7 HEADER_2x01_PARALLEL, J8 HEADER_2x01_PARALLEL, J9 HEADER_2x01_PARALLEL, M1 HOLE, M2 HOLE, M3 HOLE, M4 HOLE, U1 MICROFC-60035-SMT-TR(1), U2 OPA836IDB

Commit message: Editing schema and PCB
Parts:
- removed J1, J10, J2, J3, J7: HEADER_2x01_PARALLEL, Mlab_Pin_Headers:Straight_2x01
- added C11: 100nF, Capacitor_SMD:C_0805_2012Metric, B.Cu at (34.5, -12.2)
- added C12: 100nF, Capacitor_SMD:C_0805_2012Metric, B.Cu at (28.2, -12.2)
- added C13: 1uF/50V, Capacitor_SMD:C_0805_2012Metric, B.Cu at (25.4, -12.2)
- added C14: 10uF, Capacitor_SMD:C_0805_2012Metric, B.Cu at (30.9, -4.51)
- added C15: 10uF, Capacitor_SMD:C_0805_2012Metric, B.Cu at (33.4, -5.46)
- added D2: NSR05T40XV2T5G, Diode_SMD:D_SOD-523, B.Cu at (42.4, -13.0)
- added L1: 400uH cca 0,9mA NLV10JT391, Inductor_SMD:L_1210_3225Metric_Pad1.42x2.65mm_HandSolder, B.Cu at (45.7, -11.4)
- added R13: 100R, Resistor_SMD:R_0805_2012Metric, B.Cu at (31.2, -11.2)
- added U3: MAX5026, Package_TO_SOT_SMD:SOT-23-6_Handsoldering, B.Cu at (50.3, -10.4)
- C1: value 15uF/35V -> 10uF/35V; footprint Mlab_C:TantalC_SizeC_Reflow -> Capacitor_SMD:C_0805_2012Metric
- C10: value 0R -> 1uF/50V; footprint Mlab_R:SMD-0805 -> Capacitor_SMD:C_0805_2012Metric
- C2: value 1u5/50V - NFM41PC155B1H3L -> 10uF; footprint Mlab_L:FIR_1806 -> Capacitor_SMD:C_0805_2012Metric
- C3: value 47uF -> 10uF; footprint Mlab_C:TantalC_SizeC_Reflow -> Capacitor_SMD:C_0805_2012Metric
- C4, C7: value 10u -> 10uF; footprint Mlab_R:SMD-0805 -> Capacitor_SMD:C_0805_2012Metric
- C5, C6, C8, C9: footprint Mlab_R:SMD-0805 -> Capacitor_SMD:C_0805_2012Metric
- D1: value M4 -> BZX585-B5V6.115; footprint Mlab_D:Diode-SMA_Standard -> Diode_SMD:D_SOD-523
- R1: value 10R -> 100R; footprint Mlab_R:SMD-0805 -> Resistor_SMD:R_0805_2012Metric
- R10, R12, R2, R3, R4, R5, R8, R9: footprint Mlab_R:SMD-0805 -> Resistor_SMD:R_0805_2012Metric
- R11: value 1k -> 10k; footprint Mlab_R:SMD-0805 -> Resistor_SMD:R_0805_2012Metric
- R6: value - -> 3M9; footprint Mlab_R:SMD-0805 -> Resistor_SMD:R_0805_2012Metric
- R7: value - -> 160k; footprint Mlab_R:SMD-0805 -> Resistor_SMD:R_0805_2012Metric
- moved M2 83.1 mm to (60.0, -67.5)
- moved M1 72.4 mm to (62.5, -60.0)
- moved M3 45.6 mm to (40.0, -65.0)
- moved R6 43.0 mm to (54.4, -6.86)
- moved R7 39.7 mm to (54.4, -10.4)
- moved C2 35.1 mm to (50.0, -7.11), turned to 0 degrees
- moved J8 34.7 mm to (58.7, -5.08)
- moved J9 34.7 mm to (58.7, -2.54)
- moved J4 33.0 mm to (58.7, -10.2)
- moved J6 32.5 mm to (58.7, -12.7), turned to 0 degrees
- moved J5 32.2 mm to (58.7, -7.62), turned to 0 degrees
- moved C10 27.7 mm to (37.3, -11.9), turned to 90 degrees
- moved M4 26.4 mm to (-2.50, -55.0)
- moved C8 25.8 mm to (43.4, -4.51), turned to 90 degrees
- moved R1 23.2 mm to (22.1, -11.4), turned to 0 degrees
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Connections:
- net /#PD renamed Net-(R11-Pad2)
- C10 pad 1: /DIRECT_OUT -> Net-(C10-Pad1)
- C10 pad 2: Net-(C10-Pad2) -> GND
- C2 pad 1: Net-(C1-Pad1) -> /+3V6
- R1 pad 2: +28V -> 31V7
- R2 pad 2: Net-(C2-Pad3) -> Net-(C1-Pad1)
- R5 pad 2: Net-(C10-Pad2) -> Net-(R5-Pad2)
- R6 pad 1: Net-(R6-Pad1) -> Net-(C10-Pad1)
- R6 pad 2: /DIRECT_OUT -> /FB
- R7 pad 1: +3V3 -> /FB
- R7 pad 2: /DIRECT_OUT -> GND
- R8 pad 1: /DIRECT_OUT -> Net-(R5-Pad2)
- U1 pad 1: Net-(C10-Pad2) -> Net-(R5-Pad2)
- U1 pad 2: Net-(R6-Pad1) -> unconnected-(U1-Pad2)
- U2 pad 3: /DIRECT_OUT -> Net-(R5-Pad2)
Routing:
- net GND: track 46.9 -> 0.00 mm, vias 49 -> 0
- net /DIRECT_OUT: track 27.0 -> 0.00 mm, vias 1 -> 0
- net /+3V6: track 17.7 -> 0.00 mm
- net +3V3: track 15.4 -> 0.00 mm
- net /OUT: track 13.0 -> 0.00 mm, vias 1 -> 0
- net Net-(R11-Pad2): track 10.4 -> 0.00 mm
- net Net-(C6-Pad1): track 9.38 -> 0.00 mm, vias 1 -> 0
- net Net-(C1-Pad1): track 8.33 -> 0.00 mm
- net Net-(R10-Pad1): track 8.02 -> 0.00 mm, vias 2 -> 0
- net +28V: track 5.84 -> 0.00 mm
- net Net-(C5-Pad1): track 5.23 -> 0.00 mm
- net Net-(R10-Pad2): track 4.77 -> 0.00 mm
- net Net-(C10-Pad2): track 4.49 -> 0.00 mm, vias 1 -> 0
- net Net-(C2-Pad3): track 3.69 -> 0.00 mm
- net Net-(R6-Pad1): track 2.68 -> 0.00 mm, vias 1 -> 0
- removed copper zone on B.Cu, net GND
- removed copper zone on F.Cu, net GND
Other:
- board size 30 x 40.1 mm -> 65 x 15 mm
- board text removed: "OUT"
