File: hw/sch_pcb/USTSIPM01A.kicad_pcb (KiCad board)
At the start: 2 copper layers, 65 x 15 mm, 43 parts, among them J4 HEADER_2x01_PARALLEL, J5 HEADER_2x01_PARALLEL, J6 HEADER_2x01_PARALLEL, J8 HEADER_2x01_PARALLEL, J9 HEADER_2x01_PARALLEL, M1 HOLE, M2 HOLE, M3 HOLE, M4 HOLE, U1 MICROFC-60035-SMT-TR(1), U2 OPA836IDB, U3 MAX5026

Commit message: Editing PCB
Parts:
- removed M1, M2, M3, M4: HOLE, Mlab_Mechanical:MountingHole_3mm
- moved C8 25.7 mm to (17.8, -4.83), turned to -90 degrees
- moved D1 22.4 mm to (48.3, -5.84), turned to -90 degrees
- moved C7 20.3 mm to (20.6, -6.10), turned to -90 degrees
- moved C3 16.6 mm to (45.0, -5.59), turned to -90 degrees
- moved C14 11.0 mm to (41.9, -5.59), turned to -90 degrees
- moved R12 9.98 mm to (6.86, -2.54), turned to 90 degrees
- moved R3 7.76 mm to (32.0, -6.35), turned to 0 degrees
- moved R10 5.62 mm to (7.37, -6.20)
- moved C15 5.43 mm to (38.9, -5.59), turned to -90 degrees
- moved R6 4.02 mm to (51.1, -9.14), turned to 0 degrees
- moved J4 3.51 mm to (56.4, -7.50)
- moved J5 3.33 mm to (56.4, -10.0)
- moved C2 3.31 mm to (47.2, -8.89)
- moved R11 3.25 mm to (15.2, -4.83)
- moved U3 3.10 mm to (47.8, -12.2)
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Routing:
- net /OUT: track 0.00 -> 56.4 mm
- net /+3V6: track 0.00 -> 38.1 mm
- net Net-(C10-Pad1): track 0.00 -> 22.2 mm, vias 0 -> 2
- net +3V3: track 0.00 -> 20.4 mm
- net Net-(R5-Pad2): track 0.00 -> 13.6 mm, vias 0 -> 1
- net Net-(C6-Pad1): track 0.00 -> 10.5 mm, vias 0 -> 1
- net GND: track 0.00 -> 8.87 mm, vias 0 -> 64
- net 31V7: track 0.00 -> 7.47 mm
- net Net-(D2-Pad2): track 0.00 -> 6.58 mm
- net Net-(R10-Pad2): track 0.00 -> 6.40 mm
- net Net-(R10-Pad1): track 0.00 -> 5.21 mm
- net /FB: track 0.00 -> 4.97 mm
- net Net-(C5-Pad1): track 0.00 -> 4.78 mm
- net Net-(C1-Pad1): track 0.00 -> 4.68 mm
- net Net-(R11-Pad2): track 0.00 -> 3.36 mm
- added copper zone on B.Cu, net GND
- added copper zone on F.Cu, net GND
Other:
- board size 65 x 15 mm -> 60 x 15 mm
- board text added: "3V6"
- board text added: "OUT"
- board text added: "UST.CZ USTSIPM01A"
- board text removed: "#PD"
- board text removed: "DIROUT"
- board text removed: "IN 28V"
- board text removed: "IN 3V6"
- board text removed: "UST.CZ AIRDOSC01A_PCB01C"
