File: hw/sch_pcb/USTSIPM01A.kicad_pcb (KiCad board)
At the start: 2 copper layers, 60 x 15 mm, 39 parts, among them J4 HEADER_2x01_PARALLEL, J5 HEADER_2x01_PARALLEL, J6 HEADER_2x01_PARALLEL, J8 HEADER_2x01_PARALLEL, J9 HEADER_2x01_PARALLEL, U1 MICROFC-60035-SMT-TR(1), U2 OPA836IDB, U3 MAX5026

Commit message: Priprava vyrobnich dat
Parts:
- R8: footprint Resistor_SMD:R_0805_2012Metric -> Capacitor_SMD:C_0805_2012Metric
