File: hw/sch_pcb/USTSIPM01A.kicad_sch (KiCad schematic)
At the start: 39 parts, among them J4 HEADER_2x01_PARALLEL, J5 HEADER_2x01_PARALLEL, J6 HEADER_2x01_PARALLEL, J8 HEADER_2x01_PARALLEL, J9 HEADER_2x01_PARALLEL, U1 MICROFC-60035-SMT-TR(1), U2 OPA836IDB, U3 MAX5026

Commit message: Update title block fields.
Other:
- company: Mlab www.mlab.cz -> ust.cz
- title: SIPM02C -> USTSIPM01A
Changed lines of the file:
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@@
   (paper "A4")
   (title_block
-    (title "SIPM02C")
+    (title "USTSIPM01A")
     (date "2022-04-02")
-    (company "Mlab www.mlab.cz")
-    (comment 2 "Silicon photomultiplier interface module")
+    (company "ust.cz")
+    (comment 2 "Silicon photomultiplier\\ninterface module")
     (comment 3 "nickname <email@example.com>")
   )
